File: AccessB.kicad_pcb (KiCad board)
At the start: 2 copper layers, 50 x 62.9 mm, 30 parts, among them P1 ICSP, P2 USB_OTG, P3 GPIO, P5 USB_OTG, Q1 BSS138, Q2 BSS138, Q3 BSS138, Q4 BSS138, Q5 BSS138, U1 PIC18(L)F2550-I/SO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

Commit message: Update
PCB update in progress
Parts:
- removed MH1, MH2, MH3, MH4: DUMMY_MOUNTING-HOLE_RevE_Date22jun2010, Mounting_Holes:MountingHole_3.2mm_M3_Pad_Via
- U1: footprint SMD_Packages:SOIC-28 -> Housings_SOIC:SOIC-28W_7.5x17.9mm_Pitch1.27mm
- moved R4 149.7 mm to (45.3, 126.1)
- moved R2 149.5 mm to (42.4, 128.3)
- moved Q2 149.4 mm to (42.4, 125.7)
- moved R3 145.8 mm to (44.1, 141.8)
- moved R1 145.5 mm to (41.5, 144.5)
- moved Q1 145.5 mm to (41.4, 141.8)
- moved R10 145.0 mm to (44.8, 134.3)
- moved R7 145.0 mm to (42.0, 137.0)
- moved Q4 144.7 mm to (42.1, 134.3)
- moved R6 137.1 mm to (53.4, 128.6)
- moved Q3 136.9 mm to (53.3, 125.6)
- moved R8 136.9 mm to (56.4, 125.7)
- moved R17 125.7 mm to (66.1, 126.1)
- moved R16 125.5 mm to (63.3, 128.5)
- moved Q5 125.4 mm to (63.2, 125.7)
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Connections:
- P2 pad 4: (no net) -> Net-(P2-Pad4)
- P5 pad 2: (no net) -> Net-(P5-Pad2)
- P5 pad 3: (no net) -> Net-(P5-Pad3)
- P5 pad 4: (no net) -> Net-(P5-Pad4)
Routing:
- net GND: track 136.2 -> 0.00 mm, vias 29 -> 0
- net +5V: track 78.5 -> 0.00 mm
- net /GPIO16/RB4: track 75.5 -> 0.00 mm, vias 2 -> 0
- net /GPIO15/RB3: track 73.2 -> 0.00 mm, vias 2 -> 0
- net /VLS: track 72.2 -> 0.00 mm, vias 5 -> 0
- net /GPIO18/RB6: track 64.1 -> 0.00 mm, vias 2 -> 0
- net /GPIO17/RB5: track 61.0 -> 0.00 mm, vias 2 -> 0
- net /GPIO4/RC6: track 60.2 -> 0.00 mm, vias 1 -> 0
- net /GPIO5/RC7: track 58.1 -> 0.00 mm, vias 1 -> 0
- net /GPIO13/RB1: track 57.8 -> 0.00 mm, vias 1 -> 0
- net /GPIO19/RB7: track 56.7 -> 0.00 mm, vias 2 -> 0
- net /GPIO11/RA5: track 56.5 -> 0.00 mm
- net /GPIO12/RB0: track 53.8 -> 0.00 mm, vias 1 -> 0
- net /GPIO14/RB2: track 47.9 -> 0.00 mm, vias 1 -> 0
- net /GPIO10/RA4: track 42.7 -> 0.00 mm
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Other:
- board text removed: "1.2V"
- board text removed: "1.8V"
- board text removed: "2.5V"
- board text removed: "3.3V"
- board text removed: "VAR"
- board text removed: "VLS Voltage selector"

Commit message: Update
PCB update.
Parts:
- P5: moved to F.Cu
- moved U1 107.0 mm to (157.9, 94.5), turned to 270 degrees
- moved P1 100.4 mm to (167.6, 73.2), turned to 270 degrees
- moved P3 82.6 mm to (173.5, 112.4)
- moved P5 68.9 mm to (140.4, 83.0), turned to 270 degrees
- moved P2 47.0 mm to (140.3, 105.8)
- moved C3 46.7 mm to (146.9, 80.0)
- moved C8 44.2 mm to (156.1, 105.8), turned to 270 degrees
- moved C2 43.7 mm to (157.8, 86.2), turned to 0 degrees
- moved C4 43.3 mm to (147.2, 88.8), turned to 90 degrees
- moved C1 40.5 mm to (153.0, 86.2), turned to 180 degrees
- moved Y1 37.2 mm to (155.4, 82.2), turned to 180 degrees
Routing:
- net /GPIO16/RB4: track 0.00 -> 20.6 mm
- net /GPIO17/RB5: track 0.00 -> 14.9 mm
- net /GPIO18/RB6: track 0.00 -> 13.2 mm
- net /GPIO19/RB7: track 0.00 -> 11.1 mm
- net (no net): track 0.67 -> 0.00 mm
Other:
- board size 50 x 62.9 mm -> 50 x 50 mm
- board text removed: "Vsel"

Commit message: Updates
...
Parts:
- moved C3 36.3 mm to (113.3, 66.2)
- moved C4 36.3 mm to (113.6, 75.0)
- moved C8 11.3 mm to (167.2, 108.1)
- moved Y1 9.59 mm to (148.0, 88.4), turned to 270 degrees
- moved U1 6.64 mm to (160.8, 88.5), turned to 0 degrees
- moved C2 5.88 mm to (151.9, 86.0), turned to 90 degrees
- moved C1 4.75 mm to (151.9, 90.8), turned to 270 degrees
- moved P1 3.32 mm to (164.3, 73.5)
- moved P2 2.25 mm to (140.4, 103.5)
- moved P5 2.15 mm to (140.4, 80.9)
Connections:
- P3 pad 1: /GPIO0/RE3 -> /VLS
- P3 pad 10: /GPIO19/RB7 -> /GPIO11/RA5_VLS
- P3 pad 11: /GPIO5/RC7 -> /GPIO4/RC6
- P3 pad 12: /GPIO18/RB6 -> /GPIO3/RC2
- P3 pad 13: /GPIO6/RA0 -> /GPIO5/RC7
- P3 pad 14: /GPIO17/RB5 -> /GPIO2/RC1
- P3 pad 15: /GPIO7/RA1 -> /GPIO12/RB0
- P3 pad 16: GND -> /GPIO1/RC0
- P3 pad 17: /GPIO8/RA2 -> /GPIO13/RB1
- P3 pad 18: /GPIO15/RB3 -> /GPIO11/RA5
- P3 pad 19: /GPIO9/RA3 -> /GPIO14/RB2
- P3 pad 2: +5V -> /GPIO5/RC7_VLS
- P3 pad 20: /GPIO16/RB4 -> /GPIO10/RA4
- P3 pad 21: /GPIO10/RA4 -> /GPIO15/RB3
- P3 pad 22: /GPIO11/RA5_VLS -> /GPIO9/RA3
- P3 pad 23: /GPIO11/RA5 -> /GPIO16/RB4
- P3 pad 24: /GPIO12/RB0_VLS -> /GPIO8/RA2
- P3 pad 25: /GPIO12/RB0 -> /GPIO17/RB5
- P3 pad 26: /GPIO13/RB1_VLS -> /GPIO7/RA1
- P3 pad 27: /GPIO13/RB1 -> /GPIO18/RB6
- P3 pad 28: GND -> /GPIO6/RA0
- P3 pad 29: /GPIO14/RB2 -> /GPIO19/RB7
- P3 pad 3: /GPIO1/RC0 -> GND
- P3 pad 30: /VLS -> /GPIO0/RE3
- P3 pad 4: GND -> /GPIO4/RC6_VLS
- P3 pad 5: /GPIO2/RC1 -> GND
- P3 pad 6: /GPIO4/RC6_VLS -> /GPIO13/RB1_VLS
- P3 pad 7: /GPIO3/RC2 -> GND
- P3 pad 8: /GPIO5/RC7_VLS -> /GPIO12/RB0_VLS
- P3 pad 9: /GPIO4/RC6 -> +5V
Routing:
- net /GPIO16/RB4: track 20.6 -> 0.00 mm
- net /GPIO17/RB5: track 14.9 -> 0.00 mm
- net /GPIO18/RB6: track 13.2 -> 0.00 mm
- net /GPIO19/RB7: track 11.1 -> 0.00 mm

Commit message: Again updates
...
Parts:
- moved C8 17.2 mm to (168.2, 90.9)
- moved U1 2.05 mm to (158.8, 88.5)
- moved C1 1.15 mm to (150.8, 90.8)
- moved C2 1.15 mm to (150.8, 86.0)
- moved Y1 1.15 mm to (146.9, 88.4)
Changed lines of the file:
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@@
   (general
     (links 91)
-    (no_connects 85)
-    (area 136.524999 69.374999 186.675001 119.475001)
+    (no_connects 80)
+    (area 9.741572 30.2 274.200001 168.3774)
     (thickness 1.6)
     (drawings 74)
@@
   )
   (module Capacitors_SMD:C_0603_HandSoldering (layer F.Cu)
-    (at 151.925 90.775 270)
+    (at 150.775 90.775 270)
     (descr "Capacitor SMD 0603, hand soldering")
     (tags "capacitor 0603")
@@
   )
   (module Capacitors_SMD:C_0603_HandSoldering (layer F.Cu)
-    (at 151.925 85.975 90)
+    (at 150.775 85.975 90)
     (descr "Capacitor SMD 0603, hand soldering")
     (tags "capacitor 0603")
@@
   )
   (module Crystals:Crystal_HC49-U_Vertical (layer F.Cu)
-    (at 148.025 88.375 270)
+    (at 146.875 88.375 270)
     (descr "Crystal, Quarz, HC49/U, vertical, stehend,")
     (tags "Crystal, Quarz, HC49/U, vertical, stehend,")
@@
   )
   (module Capacitors_SMD:CP_Elec_4x5.8 (layer F.Cu)
-    (at 167.15 108.1 270)
+    (at 168.15 90.9 270)
     (descr "SMT capacitor, aluminium electrolytic, 4x5.8")
     (attr smd)
@@
   )
   (module Housings_SOIC:SOIC-28W_7.5x17.9mm_Pitch1.27mm (layer F.Cu)
-    (at 160.8 88.45)
+    (at 158.75 88.45)
     (descr "28-Lead Plastic Small Outline (SO) - Wide, 7.50 mm Body [SOIC] (see Microchip Packaging Specification 00000049BS.pdf)")
     (tags "SOIC 1.27")

Commit message: update
Parts:
- removed C8: 10uF, Capacitors_SMD:CP_Elec_4x5.8
- added C5: 100pF, Capacitors_SMD:C_0603_HandSoldering, F.Cu at (161.6, 129.5)
- moved C2 2.70 mm to (150.8, 88.7)
- moved Y1 2.70 mm to (146.9, 91.1)
- moved C1 2.70 mm to (150.8, 93.5)
Changed lines of the file:
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@@
   (general
     (links 91)
-    (no_connects 80)
-    (area 9.741572 30.2 274.200001 168.3774)
+    (no_connects 81)
+    (area 136.524999 69.374999 186.675001 119.475001)
     (thickness 1.6)
     (drawings 74)
@@
   )
   (module Capacitors_SMD:C_0603_HandSoldering (layer F.Cu)
-    (at 150.775 90.775 270)
+    (at 150.775 93.475 270)
     (descr "Capacitor SMD 0603, hand soldering")
     (tags "capacitor 0603")
@@
   )
   (module Capacitors_SMD:C_0603_HandSoldering (layer F.Cu)
-    (at 150.775 85.975 90)
+    (at 150.775 88.675 90)
     (descr "Capacitor SMD 0603, hand soldering")
     (tags "capacitor 0603")
@@
   )
   (module Crystals:Crystal_HC49-U_Vertical (layer F.Cu)
-    (at 146.875 88.375 270)
+    (at 146.875 91.075 270)
     (descr "Crystal, Quarz, HC49/U, vertical, stehend,")
     (tags "Crystal, Quarz, HC49/U, vertical, stehend,")
@@
       (net 2 GND))
   )
-  (module Capacitors_SMD:CP_Elec_4x5.8 (layer F.Cu)
-    (at 168.15 90.9 270)
-    (descr "SMT capacitor, aluminium electrolytic, 4x5.8")
-    (attr smd)
-    (fp_text reference C8 (at 0 3.54 270) (layer F.SilkS)
-      (effects (font (size 1 1) (thickness 0.15)))
-    )
-    (fp_text value 10uF (at 0 -3.54 270) (layer F.Fab)
-      (effects (font (size 1 1) (thickness 0.15)))
-    )
-    (fp_circle (center 0 0) (end 0 2) (layer F.Fab) (width 0.1))
-    (fp_text user + (at -1.12 -0.06 270) (layer F.Fab)
-      (effects (font (size 1 1) (thickness 0.15)))
-    )
-    (fp_text user + (at -2.78 2.01 270) (layer F.SilkS)
-      (effects (font (size 1 1) (thickness 0.15)))
-    )
-    (fp_text user %R (at 0 3.54 270) (layer F.Fab)
-      (effects (font (size 1 1) (thickness 0.15)))
-    )
-    (fp_line (start 2.13 2.13) (end 2.13 -2.13) (layer F.Fab) (width 0.1))
-    (fp_line (start -1.46 2.13) (end 2.13 2.13) (layer F.Fab) (width 0.1))
-    (fp_line (start -2.13 1.46) (end -1.46 2.13) (layer F.Fab) (width 0.1))
-    (fp_line (start -2.13 -1.46) (end -2.13 1.46) (layer F.Fab) (width 0.1))
-    (fp_line (start -1.46 -2.13) (end -2.13 -1.46) (layer F.Fab) (width 0.1))
-    (fp_line (start 2.13 -2.13) (end -1.46 -2.13) (layer F.Fab) (width 0.1))
-    (fp_line (start -2.29 1.52) (end -2.29 1.12) (layer F.SilkS) (width 0.12))
-    (fp_line (start 2.29 2.29) (end 2.29 1.12) (layer F.SilkS) (width 0.12))
-    (fp_line (start 2.29 -2.29) (end 2.29 -1.12) (layer F.SilkS) (width 0.12))
-    (fp_line (start -2.29 -1.52) (end -2.29 -1.12) (layer F.SilkS) (width 0.12))
-    (fp_line (start -1.52 2.29) (end 2.29 2.29) (layer F.SilkS) (width 0.12))
-    (fp_line (start -1.52 2.29) (end -2.29 1.52) (layer F.SilkS) (width 0.12))
-    (fp_line (start -1.52 -2.29) (end 2.29 -2.29) (layer F.SilkS) (width 0.12))
-    (fp_line (start -1.52 -2.29) (end -2.29 -1.52) (layer F.SilkS) (width 0.12))
-    (fp_line (start -3.35 -2.39) (end 3.35 -2.39) (layer F.CrtYd) (width 0.05))
-    (fp_line (start -3.35 -2.39) (end -3.35 2.38) (layer F.CrtYd) (width 0.05))
-    (fp_line (start 3.35 2.38) (end 3.35 -2.39) (layer F.CrtYd) (width 0.05))
-    (fp_line (start 3.35 2.38) (end -3.35 2.38) (layer F.CrtYd) (width 0.05))
-    (pad 1 smd rect (at -1.8 0 90) (size 2.6 1.6) (layers F.Cu F.Paste F.Mask)
-      (net 4 +5V))
-    (pad 2 smd rect (at 1.8 0 90) (size 2.6 1.6) (layers F.Cu F.Paste F.Mask)
-      (net 2 GND))
-    (model Capacitors_SMD.3dshapes/CP_Elec_4x5.8.wrl
-      (at (xyz 0 0 0))
-      (scale (xyz 1 1 1))
-      (rotate (xyz 0 0 180))
-    )
-  )
   (module Pin_Headers:Pin_Header_Straight_1x06_Pitch2.54mm (layer F.Cu)
     (at 164.3 73.55 270)
@@
       (at (xyz 0 0 0))
       (scale (xyz 1 1 1))
+      (rotate (xyz 0 0 0))
+    )
+  )
+  (module Capacitors_SMD:C_0603_HandSoldering (layer F.Cu)
+    (at 161.6 129.475001)
+    (descr "Capacitor SMD 0603, hand soldering")
+    (tags "capacitor 0603")
+    (attr smd)
+    (fp_text reference C5 (at 0 -1.25) (layer F.SilkS)
+      (effects (font (size 1 1) (thickness 0.15)))
+    )
+    (fp_text value 100pF (at 0 1.5) (layer F.Fab)
+      (effects (font (size 1 1) (thickness 0.15)))
+    )
+    (fp_text user %R (at 0 -1.25) (layer F.Fab)
+      (effects (font (size 1 1) (thickness 0.15)))
+    )
+    (fp_line (start -0.8 0.4) (end -0.8 -0.4) (layer F.Fab) (width 0.1))
+    (fp_line (start 0.8 0.4) (end -0.8 0.4) (layer F.Fab) (width 0.1))
+    (fp_line (start 0.8 -0.4) (end 0.8 0.4) (layer F.Fab) (width 0.1))
+    (fp_line (start -0.8 -0.4) (end 0.8 -0.4) (layer F.Fab) (width 0.1))
+    (fp_line (start -0.35 -0.6) (end 0.35 -0.6) (layer F.SilkS) (width 0.12))
+    (fp_line (start 0.35 0.6) (end -0.35 0.6) (layer F.SilkS) (width 0.12))
+    (fp_line (start -1.8 -0.65) (end 1.8 -0.65) (layer F.CrtYd) (width 0.05))
+    (fp_line (start -1.8 -0.65) (end -1.8 0.65) (layer F.CrtYd) (width 0.05))
+    (fp_line (start 1.8 0.65) (end 1.8 -0.65) (layer F.CrtYd) (width 0.05))
+    (fp_line (start 1.8 0.65) (end -1.8 0.65) (layer F.CrtYd) (width 0.05))
+    (pad 1 smd rect (at -0.95 0) (size 1.2 0.75) (layers F.Cu F.Paste F.Mask)
+      (net 4 +5V))
+    (pad 2 smd rect (at 0.95 0) (size 1.2 0.75) (layers F.Cu F.Paste F.Mask)
+      (net 2 GND))
+    (model Capacitors_SMD.3dshapes/C_0603.wrl
+      (at (xyz 0 0 0))
+      (scale (xyz 1 1 1))

Commit message: update
Parts:
- moved C3 61.9 mm to (169.1, 93.0), turned to 270 degrees
- moved C4 47.9 mm to (155.0, 99.1), turned to 0 degrees
- moved C5 38.3 mm to (165.7, 91.4), turned to 270 degrees
Routing:
- net /GPIO18/RB6: track 0.00 -> 23.8 mm
- net /GPIO19/RB7: track 0.00 -> 22.2 mm
- net /GPIO14/RB2: track 0.00 -> 11.3 mm
- net /GPIO15/RB3: track 0.00 -> 10.8 mm
- net /GPIO17/RB5: track 0.00 -> 10.4 mm
- net /GPIO16/RB4: track 0.00 -> 10.2 mm
Changed lines of the file:
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@@
   (general
     (links 91)
-    (no_connects 81)
+    (no_connects 65)
     (area 136.524999 69.374999 186.675001 119.475001)
     (thickness 1.6)
     (drawings 74)
-    (tracks 0)
+    (tracks 18)
     (zones 0)
     (modules 26)
@@
   )
   (setup
-    (last_trace_width 0.1524)
+    (last_trace_width 0.5)
     (user_trace_width 0.1524)
     (user_trace_width 0.4)
@@
   )
   (module Capacitors_SMD:CP_Elec_4x5.8 (layer F.Cu)
-    (at 113.35 66.15 90)
+    (at 169.1 92.95 270)
     (descr "SMT capacitor, aluminium electrolytic, 4x5.8")
     (attr smd)
-    (fp_text reference C3 (at -3.959 0 180) (layer F.SilkS)
-      (effects (font (size 1 1) (thickness 0.15)))
-    )
-    (fp_text value 10uF (at 0 -3.54 90) (layer F.Fab)
+    (fp_text reference C3 (at 4.3 0.05 360) (layer F.SilkS)
+      (effects (font (size 1 1) (thickness 0.15)))
+    )
+    (fp_text value 10uF (at 0 -3.54 270) (layer F.Fab)
       (effects (font (size 1 1) (thickness 0.15)))
     )
     (fp_circle (center 0 0) (end 0 2) (layer F.Fab) (width 0.1))
-    (fp_text user + (at -1.12 -0.06 90) (layer F.Fab)
-      (effects (font (size 1 1) (thickness 0.15)))
-    )
-    (fp_text user + (at -2.78 2.01 90) (layer F.SilkS)
-      (effects (font (size 1 1) (thickness 0.15)))
-    )
-    (fp_text user %R (at 0 3.54 90) (layer F.Fab)
+    (fp_text user + (at -1.12 -0.06 270) (layer F.Fab)
+      (effects (font (size 1 1) (thickness 0.15)))
+    )
+    (fp_text user + (at -2.78 2.01 270) (layer F.SilkS)
+      (effects (font (size 1 1) (thickness 0.15)))
+    )
+    (fp_text user %R (at 0 3.54 270) (layer F.Fab)
       (effects (font (size 1 1) (thickness 0.15)))
     )
@@
     (fp_line (start 3.35 2.38) (end 3.35 -2.39) (layer F.CrtYd) (width 0.05))
     (fp_line (start 3.35 2.38) (end -3.35 2.38) (layer F.CrtYd) (width 0.05))
-    (pad 1 smd rect (at -1.8 0 270) (size 2.6 1.6) (layers F.Cu F.Paste F.Mask)
+    (pad 1 smd rect (at -1.8 0 90) (size 2.6 1.6) (layers F.Cu F.Paste F.Mask)
       (net 4 +5V))
-    (pad 2 smd rect (at 1.8 0 270) (size 2.6 1.6) (layers F.Cu F.Paste F.Mask)
+    (pad 2 smd rect (at 1.8 0 90) (size 2.6 1.6) (layers F.Cu F.Paste F.Mask)
       (net 2 GND))
     (model Capacitors_SMD.3dshapes/CP_Elec_4x5.8.wrl
@@
   )
   (module Capacitors_SMD:C_0603_HandSoldering (layer F.Cu)
-    (at 113.6 75 90)
+    (at 155 99.1)
     (descr "Capacitor SMD 0603, hand soldering")
     (tags "capacitor 0603")
     (attr smd)
-    (fp_text reference C4 (at 3.1 -0.1 90) (layer F.SilkS)
-      (effects (font (size 1 1) (thickness 0.15)))
-    )
-    (fp_text value 470pF (at 18.62 43.72 90) (layer F.Fab)
+    (fp_text reference C4 (at 3.1 -0.1) (layer F.SilkS)
+      (effects (font (size 1 1) (thickness 0.15)))
+    )
+    (fp_text value 470pF (at 18.62 43.72) (layer F.Fab)
       (effects (font (size 1 1) (thickness 0.15)))
     )
@@
     (fp_line (start -0.35 -0.6) (end 0.35 -0.6) (layer F.SilkS) (width 0.15))
     (fp_line (start 0.35 0.6) (end -0.35 0.6) (layer F.SilkS) (width 0.15))
-    (pad 1 smd rect (at -0.95 0 90) (size 1.2 0.75) (layers F.Cu F.Paste F.Mask)
+    (pad 1 smd rect (at -0.95 0) (size 1.2 0.75) (layers F.Cu F.Paste F.Mask)
       (net 5 "Net-(C4-Pad1)"))
-    (pad 2 smd rect (at 0.95 0 90) (size 1.2 0.75) (layers F.Cu F.Paste F.Mask)
+    (pad 2 smd rect (at 0.95 0) (size 1.2 0.75) (layers F.Cu F.Paste F.Mask)
       (net 2 GND))
     (model Capacitors_SMD.3dshapes/C_0603_HandSoldering.wrl
@@
   )
   (module Capacitors_SMD:C_0603_HandSoldering (layer F.Cu)
-    (at 161.6 129.475001)
+    (at 165.7 91.4 270)
     (descr "Capacitor SMD 0603, hand soldering")
     (tags "capacitor 0603")
     (attr smd)
-    (fp_text reference C5 (at 0 -1.25) (layer F.SilkS)
-      (effects (font (size 1 1) (thickness 0.15)))
-    )
-    (fp_text value 100pF (at 0 1.5) (layer F.Fab)
-      (effects (font (size 1 1) (thickness 0.15)))
-    )
-    (fp_text user %R (at 0 -1.25) (layer F.Fab)
+    (fp_text reference C5 (at -2.95 -0.05 450) (layer F.SilkS)
+      (effects (font (size 1 1) (thickness 0.15)))
+    )
+    (fp_text value 100pF (at 0 1.5 270) (layer F.Fab)
+      (effects (font (size 1 1) (thickness 0.15)))
+    )
+    (fp_text user %R (at 0 -1.25 270) (layer F.Fab)
       (effects (font (size 1 1) (thickness 0.15)))
     )
@@
     (fp_line (start 1.8 0.65) (end 1.8 -0.65) (layer F.CrtYd) (width 0.05))
     (fp_line (start 1.8 0.65) (end -1.8 0.65) (layer F.CrtYd) (width 0.05))
-    (pad 1 smd rect (at -0.95 0) (size 1.2 0.75) (layers F.Cu F.Paste F.Mask)
+    (pad 1 smd rect (at -0.95 0 270) (size 1.2 0.75) (layers F.Cu F.Paste F.Mask)
       (net 4 +5V))
-    (pad 2 smd rect (at 0.95 0) (size 1.2 0.75) (layers F.Cu F.Paste F.Mask)
+    (pad 2 smd rect (at 0.95 0 270) (size 1.2 0.75) (layers F.Cu F.Paste F.Mask)
       (net 2 GND))
     (model Capacitors_SMD.3dshapes/C_0603.wrl
@@
   (gr_line (start 186.6 119.4) (end 136.6 119.4) (angle 90) (layer Edge.Cuts) (width 0.15))
   (gr_line (start 136.6 69.45) (end 186.6 69.45) (angle 90) (layer Edge.Cuts) (width 0.15))
+  (segment (start 156.68 73.55) (end 156.68 75.68) (width 0.5) (layer F.Cu) (net 7) (status 400000))
+  (segment (start 161.195 80.195) (end 163.45 80.195) (width 0.5) (layer F.Cu) (net 7) (status 800000))
+  (segment (start 156.68 75.68) (end 161.195 80.195) (width 0.5) (layer F.Cu) (net 7))
+  (segment (start 163.45 80.195) (end 170.135 80.195) (width 0.5) (layer F.Cu) (net 7))
+  (segment (start 170.135 80.195) (end 173.51 76.82) (width 0.5) (layer F.Cu) (net 7))
+  (segment (start 154.14 73.55) (end 154.14 74.09) (width 0.5) (layer F.Cu) (net 8) (status C00000))
+  (segment (start 154.14 74.09) (end 161.515 81.465) (width 0.5) (layer F.Cu) (net 8) (status 400000))
+  (segment (start 161.515 81.465) (end 163.45 81.465) (width 0.5) (layer F.Cu) (net 8) (status 800000))
+  (segment (start 163.45 81.465) (end 171.405 81.465) (width 0.5) (layer F.Cu) (net 8))
+  (segment (start 171.405 81.465) (end 173.51 79.36) (width 0.5) (layer F.Cu) (net 8))
+  (segment (start 163.45 82.735) (end 172.675 82.735) (width 0.5) (layer F.Cu) (net 19))
+  (segment (start 172.675 82.735) (end 173.51 81.9) (width 0.5) (layer F.Cu) (net 19))
+  (segment (start 163.45 85.275) (end 171.805 85.275) (width 0.5) (layer F.Cu) (net 20))
+  (segment (start 171.805 85.275) (end 173.51 86.98) (width 0.5) (layer F.Cu) (net 20))
+  (segment (start 163.45 86.545) (end 170.535 86.545) (width 0.5) (layer F.Cu) (net 21))
+  (segment (start 170.535 86.545) (end 173.51 89.52) (width 0.5) (layer F.Cu) (net 21))
+  (segment (start 163.45 84.005) (end 173.075 84.005) (width 0.5) (layer F.Cu) (net 22))
+  (segment (start 173.075 84.005) (end 173.51 84.44) (width 0.5) (layer F.Cu) (net 22))
   (zone (net 2) (net_name GND) (layer F.Cu) (hatch edge 0.508)
     (connect_pads (clearance 0.508))

Commit message: update again
Routing:
- net /GPIO3/RC2: track 0.00 -> 26.7 mm, vias 0 -> 1
- net /GPIO11/RA5: track 0.00 -> 26.3 mm, vias 0 -> 1
- net /GPIO2/RC1: track 0.00 -> 25.8 mm, vias 0 -> 1
- net /GPIO1/RC0: track 0.00 -> 25.3 mm, vias 0 -> 1
- net /GPIO0/RE3: track 0.00 -> 24.8 mm, vias 0 -> 1
- net /GPIO6/RA0: track 0.00 -> 24.0 mm, vias 0 -> 1
- net /GPIO10/RA4: track 0.00 -> 23.7 mm, vias 0 -> 1
- net /GPIO7/RA1: track 0.00 -> 23.4 mm, vias 0 -> 1
- net /GPIO9/RA3: track 0.00 -> 23.2 mm, vias 0 -> 1
- net /GPIO8/RA2: track 0.00 -> 22.8 mm, vias 0 -> 1
- net /GPIO12/RB0: track 0.00 -> 14.4 mm
- net /GPIO4/RC6: track 0.00 -> 13.4 mm
- net /GPIO5/RC7: track 0.00 -> 12.8 mm
- net /GPIO13/RB1: track 0.00 -> 12.7 mm
- net Net-(C1-Pad1): track 0.00 -> 7.96 mm
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
Commit message: another upd
Parts:
- added C6: 10uF, Capacitors_SMD:CP_Elec_4x5.8, F.Cu at (146.2, 100.4)
- added C7: 10uF, Capacitors_SMD:CP_Elec_4x5.8, F.Cu at (147.8, 81.0)
- added C8: 100pF, Capacitors_SMD:C_0603_HandSoldering, F.Cu at (154.9, 114.5)
- added C9: 100pF, Capacitors_SMD:C_0603_HandSoldering, F.Cu at (144.3, 80.5)
Routing:
- net /GPIO0/RE3: track 24.8 -> 30.6 mm
