File: AccessB.kicad_pcb (KiCad board)
At the start: 2 copper layers, 50 x 50 mm, 30 parts, among them Q1 BSS138, Q2 BSS138, Q3 BSS138, Q4 BSS138, Q5 BSS138, U1 PIC18(L)F2550-I/SO, Y1 4MHz

Commit message: updat
Other:
- board text added: "PIC18F2550 SOIC28-W"
- board text removed: "****NOTA IPORTANTE: Cambiar empaquetado del PIC de SOIC-28-Narrow a SOIC-28-Wide"
- board text removed: "**Cambiar la selección de voltage usando jumpers por DIP switch"
- board text removed: "**Mover C3 por que pega con el Pickit cuando es insertado"
- board text removed: "+5V"
- board text removed: "- P2 es para alimentacion/USB"
- board text removed: "-Acomodar mejor las notas de componentes de la circuiteria del VLC"
- board text removed: "-Indicar que el P1 es el ICSP"
- board text removed: "-P5 es puerto para alimentacon solamente"
- board text removed: "Afortunadamente doblando los pines del PIC hacia abajo como si fuera un SOJ-28 encaja perfecto en el empaquetado del SOIC-28-Narrow"
- board text removed: "GPIO0"
- board text removed: "ya que el empaquetado del PIC es SOIC-28-Wide y por error en el diseño que envie a PCBway va con SOIC-28-Narrow"

Commit message: Maybe the final version...
Maybe....??
Routing:
- net GND: vias 122 -> 116
- net +5V: vias 6 -> 3
Other:
- board text added: "+5V"
- board text added: "+VLS"
- board text added: "A0/IO06"
- board text added: "A4/IO10"
- board text added: "ANALOG IN: AN0-A0 AN1-A1 AN2-A2 AN3-A3 AN4-A5 AN8-B2 AN9-B3 AN10-B1 AN11-B4 AN12-B0"
- board text added: "AccessB V2 OTrevizo"
- board text added: "C0/IO01"
- board text added: "C1/IO02"
- board text added: "C2/IO03"
- board text added: "CCP MODULE PINOUT: C1/CCP2 C2/CCP1"
- board text added: "CTS/A3/IO09"
- board text added: "DTR/A1/IO07"
- board text added: "E3/IO00"
- board text added: "GND"
- board text added: "IO12/SDA/SDI/B0"
- board text added: "IO13/SCK/SCL/B1"
- board text added: "IO14/B2"
- board text added: "IO15/B3"
- board text added: "IO16/DTS/B4"
- board text added: "IO17/B5"
- board text added: "IO18/B6"
- board text added: "IO19/B7"
- board text added: "IO4/TX/CK/C6"
- board text added: "IO5/RX/DT/SDO/C7"
- board text added: "RTS/A2/IO08"
- board text added: "RX/SDO VLS_IO5"
- board text added: "SCK/SCL VLS_IO13"
- board text added: "SDA/SDI VLS_IO12"
- board text added: "TX/VLS_IO4"
- board text added: "_SS/A5/IO11"
- board text added: "_SS/VLS_IO11"
- board text removed: "***Agregar mejores notas del silkscreen tomando en cuenta la siguiente lista:"
- board text removed: "-Colocar mejor la numeracion de los GPIO en el P3, si es posible por ambas caras del PCB"
- board text removed: "-Indicar las lineas de CTS/RTS/DTR/DSR"
- board text removed: "-Tabla de GPIO que incluya tambien funciones básicas del pin y puerto"
