File: AccessB.sch (KiCad schematic (older format))
At the start: 15 parts, among them P1 ICSP, P2 USB_OTG, P3 GPIO, P5 USB_OTG, U1 PIC18(L)F2550-I/SO, Y1 4MHz

Commit message: Update
PCB update in progress
Parts:
- removed MH1, MH2, MH3, MH4: DUMMY_MOUNTING-HOLE_RevE_Date22jun2010, Mounting_Holes:MountingHole_3.2mm_M3_Pad_Via, symbol DUMMY_MOUNTING-HOLE_RevE_Date22jun2010
- U1: footprint SMD_Packages:SOIC-28 -> Housings_SOIC:SOIC-28W_7.5x17.9mm_Pitch1.27mm
Changed lines of the file:
@@
 F 0 "U1" H 3650 3700 50  0000 C CNN
 F 1 "PIC18(L)F2550-I/SO" H 5300 1700 50  0000 C CNN
-F 2 "SMD_Packages:SOIC-28" H 4650 2700 50  0000 C CIN
+F 2 "Housings_SOIC:SOIC-28W_7.5x17.9mm_Pitch1.27mm" H 4650 2700 50  0000 C CIN
 F 3 "" H 4650 2250 60  0000 C CNN
 	1    4650 2700
@@
 	1    0    0    -1
 $EndComp
-$Comp
-L DUMMY_MOUNTING-HOLE_RevE_Date22jun2010 MH1
-U 1 1 5B4C541A
-P 1500 7300
-F 0 "MH1" H 1500 7500 50  0000 C CNN
-F 1 "DUMMY_MOUNTING-HOLE_RevE_Date22jun2010" H 1500 7100 50  0000 C CNN
-F 2 "Mounting_Holes:MountingHole_3.2mm_M3_Pad_Via" H 1500 7300 50  0001 C CNN
-F 3 "" H 1500 7300 50  0000 C CNN
-	1    1500 7300
-	1    0    0    -1
-$EndComp
-$Comp
-L DUMMY_MOUNTING-HOLE_RevE_Date22jun2010 MH3
-U 1 1 5B4C54EF
-P 3400 7300
-F 0 "MH3" H 3400 7500 50  0000 C CNN
-F 1 "DUMMY_MOUNTING-HOLE_RevE_Date22jun2010" H 3400 7100 50  0000 C CNN
-F 2 "Mounting_Holes:MountingHole_3.2mm_M3_Pad_Via" H 3400 7300 50  0001 C CNN
-F 3 "" H 3400 7300 50  0000 C CNN
-	1    3400 7300
-	1    0    0    -1
-$EndComp
-$Comp
-L DUMMY_MOUNTING-HOLE_RevE_Date22jun2010 MH4
-U 1 1 5B4C55A8
-P 5300 7300
-F 0 "MH4" H 5300 7500 50  0000 C CNN
-F 1 "DUMMY_MOUNTING-HOLE_RevE_Date22jun2010" H 5300 7100 50  0000 C CNN
-F 2 "Mounting_Holes:MountingHole_3.2mm_M3_Pad_Via" H 5300 7300 50  0001 C CNN
-F 3 "" H 5300 7300 50  0000 C CNN
-	1    5300 7300
-	1    0    0    -1
-$EndComp
-$Comp
-L DUMMY_MOUNTING-HOLE_RevE_Date22jun2010 MH2
-U 1 1 5B4C5658
-P 3400 6600
-F 0 "MH2" H 3400 6800 50  0000 C CNN
-F 1 "DUMMY_MOUNTING-HOLE_RevE_Date22jun2010" H 3400 6400 50  0000 C CNN
-F 2 "Mounting_Holes:MountingHole_3.2mm_M3_Pad_Via" H 3400 6600 50  0001 C CNN
-F 3 "" H 3400 6600 50  0000 C CNN
-	1    3400 6600
-	1    0    0    -1
-$EndComp
-Text GLabel 3750 6600 2    60   UnSpc ~ 0
-GND
-Text GLabel 3750 7300 2    60   UnSpc ~ 0
-GND
-Text GLabel 5650 7300 2    60   UnSpc ~ 0
-GND
-Text GLabel 1800 7300 2    60   UnSpc ~ 0
-GND
 Wire Wire Line
 	1650 2500 1650 3250
@@
 	5200 5550 5200 5750
 Connection ~ 5200 5750
-Wire Wire Line
-	3750 6600 3400 6600
-Wire Wire Line
-	1800 7300 1500 7300
-Wire Wire Line
-	3750 7300 3400 7300
-Wire Wire Line
-	5650 7300 5300 7300
 $EndSCHEMATC

Commit message: Updates
...
Connections:
- net GND: now also P3.3 (P3), P3.5 (P5), P3.7 (P7); no longer P3.16 (P16), P3.28 (P28), P3.4 (P4)
- net GPIO0/RE3: now also P3.30 (P30); no longer P3.1 (P1)
- net GPIO1/RC0: now also P3.16 (P16); no longer P3.3 (P3)
- net GPIO10/RA4: now also P3.20 (P20); no longer P3.21 (P21)
- net GPIO11/RA5: now also P3.18 (P18); no longer P3.23 (P23)
- net GPIO11/RA5_VLS: now also P3.10 (P10); no longer P3.22 (P22)
- net GPIO12/RB0: now also P3.15 (P15); no longer P3.25 (P25)
- net GPIO12/RB0_VLS: now also P3.8 (P8); no longer P3.24 (P24)
- net GPIO13/RB1: now also P3.17 (P17); no longer P3.27 (P27)
- net GPIO13/RB1_VLS: now also P3.6 (P6); no longer P3.26 (P26)
- net GPIO14/RB2: now also P3.19 (P19); no longer P3.29 (P29)
- net GPIO15/RB3: now also P3.21 (P21); no longer P3.18 (P18)
- net GPIO16/RB4: now also P3.23 (P23); no longer P3.20 (P20)
- net GPIO17/RB5: now also P3.25 (P25); no longer P3.14 (P14)
- net GPIO18/RB6: now also P3.27 (P27); no longer P3.12 (P12)
- net GPIO19/RB7: now also P3.29 (P29); no longer P3.10 (P10)
- net GPIO2/RC1: now also P3.14 (P14); no longer P3.5 (P5)
- net GPIO3/RC2: now also P3.12 (P12); no longer P3.7 (P7)
- net GPIO4/RC6: now also P3.11 (P11); no longer P3.9 (P9)
- net GPIO4/RC6_VLS: now also P3.4 (P4); no longer P3.6 (P6)
- net GPIO5/RC7: now also P3.13 (P13); no longer P3.11 (P11)
- net GPIO5/RC7_VLS: now also P3.2 (P2); no longer P3.8 (P8)
- net GPIO6/RA0: now also P3.28 (P28); no longer P3.13 (P13)
- net GPIO7/RA1: now also P3.26 (P26); no longer P3.15 (P15)
- net GPIO8/RA2: now also P3.24 (P24); no longer P3.17 (P17)
- net GPIO9/RA3: now also P3.22 (P22); no longer P3.19 (P19)
- net VCC: now also P3.9 (P9); no longer P3.2 (P2)
- net VLS: now also P3.1 (P1); no longer P3.30 (P30)
Changed lines of the file:
@@
 	1    0    0    -1
 $EndComp
-Text Label 8400 1250 2    60   ~ 0
-GPIO1/RC0
+Text Label 8900 1650 0    60   ~ 0
+GPIO3/RC2
+Text Label 8400 1650 2    60   ~ 0
+GPIO4/RC6
+Text Label 8400 1750 2    60   ~ 0
+GPIO5/RC7
+Text Label 8900 2450 0    60   ~ 0
+GPIO6/RA0
+Text Label 8900 2350 0    60   ~ 0
+GPIO7/RA1
+Text Label 8900 2250 0    60   ~ 0
+GPIO8/RA2
+Text Label 8900 2150 0    60   ~ 0
+GPIO9/RA3
+Text Label 8900 2050 0    60   ~ 0
+GPIO10/RA4
+Text Label 8900 1950 0    60   ~ 0
+GPIO11/RA5
+Text Label 8400 1850 2    60   ~ 0
+GPIO12/RB0
+Text Label 8400 1950 2    60   ~ 0
+GPIO13/RB1
+Text Label 8400 2050 2    60   ~ 0
+GPIO14/RB2
+Text Label 8400 2150 2    60   ~ 0
+GPIO15/RB3
+Text Label 8400 2250 2    60   ~ 0
+GPIO16/RB4
+Text Label 8400 2350 2    60   ~ 0
+GPIO17/RB5
+Text Label 8400 2450 2    60   ~ 0
+GPIO18/RB6
+Text Label 8400 2550 2    60   ~ 0
+GPIO19/RB7
+Text Label 8900 1250 0    60   ~ 0
+GPIO4/RC6_VLS
+Text Label 8900 1150 0    60   ~ 0
+GPIO5/RC7_VLS
+Text Label 8900 1550 0    60   ~ 0
+GPIO11/RA5_VLS
+Text Label 8900 1450 0    60   ~ 0
+GPIO12/RB0_VLS
+Text Label 8900 1350 0    60   ~ 0
+GPIO13/RB1_VLS
+Text Label 8400 1550 2    60   ~ 0
++5V
 Text Label 8400 1350 2    60   ~ 0
-GPIO2/RC1
-Text Label 8400 1450 2    60   ~ 0
-GPIO3/RC2
-Text Label 8400 1550 2    60   ~ 0
-GPIO4/RC6
-Text Label 8400 1650 2    60   ~ 0
-GPIO5/RC7
-Text Label 8400 1750 2    60   ~ 0
-GPIO6/RA0
-Text Label 8400 1850 2    60   ~ 0
-GPIO7/RA1
-Text Label 8400 1950 2    60   ~ 0
-GPIO8/RA2
-Text Label 8400 2050 2    60   ~ 0
-GPIO9/RA3
-Text Label 8400 2150 2    60   ~ 0
-GPIO10/RA4
-Text Label 8400 2250 2    60   ~ 0
-GPIO11/RA5
-Text Label 8400 2350 2    60   ~ 0
-GPIO12/RB0
-Text Label 8400 2450 2    60   ~ 0
-GPIO13/RB1
-Text Label 8400 2550 2    60   ~ 0
-GPIO14/RB2
-Text Label 8900 1950 0    60   ~ 0
-GPIO15/RB3
-Text Label 8900 2050 0    60   ~ 0
-GPIO16/RB4
-Text Label 8900 1750 0    60   ~ 0
-GPIO17/RB5
-Text Label 8900 1650 0    60   ~ 0
-GPIO18/RB6
-Text Label 8900 1550 0    60   ~ 0
-GPIO19/RB7
-Text Label 8900 1350 0    60   ~ 0
-GPIO4/RC6_VLS
-Text Label 8900 1450 0    60   ~ 0
-GPIO5/RC7_VLS
-Text Label 8900 2150 0    60   ~ 0
-GPIO11/RA5_VLS
-Text Label 8900 2250 0    60   ~ 0
-GPIO12/RB0_VLS
-Text Label 8900 2350 0    60   ~ 0
-GPIO13/RB1_VLS
-Text Label 8900 1150 0    60   ~ 0
-+5V
-Text Label 8900 1250 0    60   ~ 0
 GND
 $Comp
@@
 Text Label 5850 2900 0    60   ~ 0
 GPIO0/RE3
-Text Label 8400 1150 2    60   ~ 0
+Text Label 8900 2550 0    60   ~ 0
 GPIO0/RE3
 Entry Wire Line
@@
 	7700 1950 7800 2050
 Entry Wire Line
-	7700 2050 7800 2150
-Entry Wire Line
 	7700 2150 7800 2250
 Entry Wire Line
@@
 Entry Wire Line
 	6400 2900 6500 3000
-Text Label 6200 1000 0    118  ~ 24
+Text Label 5650 1000 0    118  ~ 24
 GPIO_BUS
 Text Notes 3350 5000 0    118  ~ 24
@@
 Text Notes 1450 5000 0    118  ~ 24
 ICSP HEADER
-Text Label 8900 2450 0    60   ~ 0
+Text Label 8400 1250 2    60   ~ 0
 GND
 $Comp
@@
 Text GLabel 4650 1400 1    60   UnSpc ~ 0
 +5V
-Text Label 8900 2550 0    60   ~ 0
+Text Label 8400 1150 2    60   ~ 0
 VLS
-Text Label 8900 1850 0    60   ~ 0
+Text Label 8400 1450 2    60   ~ 0
 GND
 $Comp
@@
 	9800 1000 9800 2450
 Wire Wire Line
-	7800 1150 8400 1150
-Wire Wire Line
-	7800 1250 8400 1250
-Wire Wire Line
-	7800 1350 8400 1350
-Wire Wire Line
-	7800 1450 8400 1450
-Wire Wire Line
-	7800 1550 8400 1550
-Wire Wire Line
-	7800 1650 8400 1650
-Wire Wire Line
-	7800 1750 8400 1750
-Wire Wire Line
-	7800 1850 8400 1850
-Wire Wire Line
-	7800 1950 8400 1950
-Wire Wire Line
-	7800 2050 8400 2050
-Wire Wire Line
-	7800 2150 8400 2150
-Wire Wire Line
 	7800 2250 8400 2250
 Wire Wire Line
@@
 	5200 5550 5200 5750
 Connection ~ 5200 5750
+Text Label 8900 1750 0    60   ~ 0
+GPIO2/RC1
+Text Label 8900 1850 0    60   ~ 0
+GPIO1/RC0
+Entry Wire Line
+	7700 2050 7800 2150
+Wire Wire Line
+	7800 2150 8400 2150
+Wire Wire Line
+	7800 2050 8400 2050
+Wire Wire Line
+	7800 1950 8400 1950
+Wire Wire Line
+	7800 1850 8400 1850
+Wire Wire Line
+	7800 1750 8400 1750
+Wire Wire Line
+	7800 1650 8400 1650
+Wire Wire Line
+	7800 1550 8400 1550
+Wire Wire Line
+	7800 1450 8400 1450
+Wire Wire Line
+	7800 1350 8400 1350
+Wire Wire Line
+	7800 1250 8400 1250
+Wire Wire Line
+	7800 1150 8400 1150
 $EndSCHEMATC

Commit message: Again updates
...
Parts:
- removed C8: 10uF, Capacitors_SMD:CP_Elec_4x5.8, symbol CP
- added C5: 100pF, Capacitors_SMD:C_0603_HandSoldering, symbol C
Connections:
- net VCC is gone; now on net GND: C3.1, P1.2 (P2), P2.1 (VCC), P3.9 (P9), P5.1 (VCC), U1.20 (VDD)
- net GND: now also C5.1, C5.2
Other:
- note added: "IC DECOUPLING"
- note added: "USB POWER"
- moved on the sheet: C3, P5
Changed lines of the file:
@@
 L CP C3
 U 1 1 5629C0F8
-P 3050 5450
-F 0 "C3" H 3075 5550 50  0000 L CNN
-F 1 "10uF" H 3075 5350 50  0000 L CNN
-F 2 "Capacitors_SMD:CP_Elec_4x5.8" H 3088 5300 30  0001 C CNN
-F 3 "" H 3050 5450 60  0000 C CNN
-	1    3050 5450
+P 6900 5600
+F 0 "C3" H 6925 5700 50  0000 L CNN
+F 1 "10uF" H 6925 5500 50  0000 L CNN
+F 2 "Capacitors_SMD:CP_Elec_4x5.8" H 6938 5450 30  0001 C CNN
+F 3 "" H 6900 5600 60  0000 C CNN
+	1    6900 5600
 	1    0    0    -1
 $EndComp
@@
 L GND #PWR01
 U 1 1 5632DC45
-P 6750 5400
-F 0 "#PWR01" H 6750 5150 50  0001 C CNN
-F 1 "GND" H 6750 5250 50  0000 C CNN
-F 2 "" H 6750 5400 60  0000 C CNN
-F 3 "" H 6750 5400 60  0000 C CNN
-	1    6750 5400
+P 2150 6750
+F 0 "#PWR01" H 2150 6500 50  0001 C CNN
+F 1 "GND" H 2150 6600 50  0000 C CNN
+F 2 "" H 2150 6750 60  0000 C CNN
+F 3 "" H 2150 6750 60  0000 C CNN
+	1    2150 6750
 	1    0    0    -1
 $EndComp
@@
 L PWR_FLAG #FLG03
 U 1 1 56332B13
-P 6750 5200
-F 0 "#FLG03" H 6750 5295 50  0001 C CNN
-F 1 "PWR_FLAG" H 6750 5380 50  0000 C CNN
-F 2 "" H 6750 5200 60  0000 C CNN
-F 3 "" H 6750 5200 60  0000 C CNN
-	1    6750 5200
+P 2150 6550
+F 0 "#FLG03" H 2150 6645 50  0001 C CNN
+F 1 "PWR_FLAG" H 2150 6730 50  0000 C CNN
+F 2 "" H 2150 6550 60  0000 C CNN
+F 3 "" H 2150 6550 60  0000 C CNN
+	1    2150 6550
 	1    0    0    -1
 $EndComp
@@
 	1    0    0    -1
 $EndComp
-Text GLabel 6950 5300 2    60   UnSpc ~ 0
+Text GLabel 2350 6650 2    60   UnSpc ~ 0
 GND
 Text GLabel 3050 5000 1    60   UnSpc ~ 0
@@
 L USB_OTG-RESCUE-AccessB P5
 U 1 1 592BE443
-P 5850 5350
-F 0 "P5" H 6175 5225 50  0000 C CNN
-F 1 "USB_OTG" H 5850 5550 50  0000 C CNN
-F 2 "Connect:USB_Micro-B" V 5800 5250 60  0001 C CNN
-F 3 "" V 5800 5250 60  0000 C CNN
-	1    5850 5350
+P 5350 5350
+F 0 "P5" H 5675 5225 50  0000 C CNN
+F 1 "USB_OTG" H 5350 5550 50  0000 C CNN
+F 2 "Connect:USB_Micro-B" V 5300 5250 60  0001 C CNN
+F 3 "" V 5300 5250 60  0000 C CNN
+	1    5350 5350
 	0    1    1    0
 $EndComp
-Text GLabel 5200 5050 1    60   UnSpc ~ 0
+Text GLabel 4700 5050 1    60   UnSpc ~ 0
 +5V
-$Comp
-L CP C8
-U 1 1 592BE632
-P 5200 5400
-F 0 "C8" H 5225 5500 50  0000 L CNN
-F 1 "10uF" H 5225 5300 50  0000 L CNN
-F 2 "Capacitors_SMD:CP_Elec_4x5.8" H 5238 5250 30  0001 C CNN
-F 3 "" H 5200 5400 60  0000 C CNN
-	1    5200 5400
-	1    0    0    -1
-$EndComp
-NoConn ~ 5550 5450
-NoConn ~ 5550 5350
-NoConn ~ 5550 5250
+NoConn ~ 5050 5450
+NoConn ~ 5050 5350
+NoConn ~ 5050 5250
 $Comp
 L PWR_FLAG #FLG07
@@
 	1    0    0    -1
 $EndComp
-Wire Wire Line
-	1650 2500 1650 3250
-Wire Wire Line
-	1650 2900 1800 2900
-Wire Wire Line
-	2250 2600 2250 3250
-Wire Wire Line
-	2250 2900 2100 2900
-Wire Wire Line
-	1650 3550 1650 3750
-Wire Wire Line
-	1650 3750 2250 3750
-Wire Wire Line
-	2250 3750 2250 3550
-Wire Wire Line
-	1950 3900 1950 3750
-Connection ~ 1950 3750
-Wire Wire Line
-	4550 3800 4550 4000
-Wire Wire Line
-	4550 4000 4650 4000
-Wire Wire Line
-	4650 4000 4650 3800
-Connection ~ 4600 4000
-Wire Wire Line
-	6750 5200 6750 5400
-Wire Wire Line
-	4650 1600 4650 1400
-Wire Wire Line
-	3050 5000 3050 5300
-Wire Wire Line
-	2900 5150 3900 5150
-Wire Wire Line
-	3900 5550 3750 5550
-Wire Wire Line
-	3750 5550 3750 5850
-Wire Wire Line
-	3050 5750 5950 5750
-Connection ~ 3750 5750
-Connection ~ 3050 5150
-Wire Wire Line
-	3050 5600 3050 5750
-Wire Wire Line
-	3450 2500 1650 2500
-Connection ~ 1650 2900
-Wire Wire Line
-	3450 2600 2250 2600
-Connection ~ 2250 2900
-Wire Wire Line
-	5850 2700 6800 2700
-Wire Wire Line
-	6800 2700 6800 2900
-Wire Wire Line
-	6800 3200 6800 3400
-Wire Bus Line
-	2800 1000 2800 2300
-Wire Bus Line
-	2800 1000 9800 1000
-Wire Bus Line
-	7700 1000 7700 4400
-Wire Bus Line
-	6450 1000 6450 2400
-Wire Bus Line
-	2800 2900 2800 4400
-Wire Bus Line
-	2800 4400 7700 4400
-Wire Bus Line
-	9800 1000 9800 2450
-Wire Wire Line
-	7800 2250 8400 2250
-Wire Wire Line
-	7800 2350 8400 2350
-Wire Wire Line
-	7800 2450 8400 2450
-Wire Wire Line
-	7800 2550 8400 2550
-Wire Bus Line
-	6500 3000 6500 4400
-Wire Wire Line
-	5850 2900 6400 2900
-Wire Wire Line
-	5850 1900 6350 1900
-Wire Wire Line
-	5850 2000 6350 2000
-Wire Wire Line
-	5850 2100 6350 2100
-Wire Wire Line
-	5850 2400 6350 2400
-Wire Wire Line
-	5850 2500 6350 2500
-Wire Wire Line
-	2900 1900 3450 1900
-Wire Wire Line
-	2900 2000 3450 2000
-Wire Wire Line
-	2900 2100 3450 2100
-Wire Wire Line
-	2900 2200 3450 2200
-Wire Wire Line
-	2900 2300 3450 2300
-Wire Wire Line
-	2900 2400 3450 2400
-Wire Wire Line
-	2900 2800 3450 2800
-Wire Wire Line
-	2900 2900 3450 2900
-Wire Wire Line
-	2900 3000 3450 3000
-Wire Wire Line
-	2900 3100 3450 3100
-Wire Wire Line
-	2900 3200 3450 3200
-Wire Wire Line
-	2900 3300 3450 3300
-Wire Wire Line
-	2900 3400 3450 3400
-Wire Wire Line
-	2900 3500 3450 3500
-Wire Wire Line
-	6950 5300 6750 5300
-Connection ~ 6750 5300
-Wire Wire Line
-	9050 3400 9300 3400
-Wire Wire Line
-	9050 3550 9300 3550
-Wire Wire Line
-	9050 3700 9300 3700
-Wire Wire Line
-	9050 3850 9300 3850
-Wire Wire Line
-	9050 4000 9300 4000
-Wire Wire Line
-	9050 4350 9300 4350
-Wire Wire Line
-	9050 4500 9300 4500
-Wire Wire Line
-	9050 4650 9300 4650
-Wire Wire Line
-	9050 4800 9300 4800
-Wire Wire Line
-	9050 4950 9300 4950
-Wire Wire Line
-	9050 4150 9300 4150
-Wire Wire Line
-	5200 5250 5200 5050
-Wire Wire Line
-	5550 5150 5200 5150
-Connection ~ 5200 5150
-Wire Wire Line
-	3250 4800 3250 5150
-Connection ~ 3250 5150
-Wire Wire Line
-	2900 4900 2900 5150
-Connection ~ 4300 5750
-Wire Wire Line
-	5550 5550 5550 5750
-Connection ~ 5550 5750
-Wire Wire Line
-	5200 5550 5200 5750
-Connection ~ 5200 5750
 Text Label 8900 1750 0    60   ~ 0
 GPIO2/RC1
@@
 	7700 2050 7800 2150
 Wire Wire Line
+	1650 2500 1650 3250
+Wire Wire Line
+	1650 2900 1800 2900
+Wire Wire Line
+	2250 2600 2250 3250
+Wire Wire Line
+	2250 2900 2100 2900
+Wire Wire Line
+	1650 3550 1650 3750
+Wire Wire Line
+	1650 3750 2250 3750
+Wire Wire Line
+	2250 3750 2250 3550
+Wire Wire Line
+	1950 3900 1950 3750
+Connection ~ 1950 3750
+Wire Wire Line
+	4550 3800 4550 4000
+Wire Wire Line
+	4550 4000 4650 4000
+Wire Wire Line
+	4650 4000 4650 3800
+Connection ~ 4600 4000
+Wire Wire Line
+	2150 6550 2150 6750
+Wire Wire Line
+	4650 1600 4650 1400
+Wire Wire Line
+	3050 5000 3050 5750
+Wire Wire Line
+	2900 5150 3900 5150
+Wire Wire Line
+	3900 5550 3750 5550
+Wire Wire Line
+	3750 5550 3750 5850
+Connection ~ 3750 5750
+Connection ~ 3050 5150
+Wire Wire Line
+	3450 2500 1650 2500
+Connection ~ 1650 2900
+Wire Wire Line
+	3450 2600 2250 2600
+Connection ~ 2250 2900
+Wire Wire Line
+	5850 2700 6800 2700
+Wire Wire Line
+	6800 2700 6800 2900
+Wire Wire Line
+	6800 3200 6800 3400
+Wire Bus Line
+	2800 1000 2800 2300
+Wire Bus Line
+	2800 1000 9800 1000
+Wire Bus Line
+	7700 1000 7700 4400
+Wire Bus Line
+	6450 1000 6450 2400
+Wire Bus Line
+	2800 2900 2800 4400
+Wire Bus Line
+	2800 4400 7700 4400
+Wire Bus Line
+	9800 1000 9800 2450
+Wire Wire Line
+	7800 2250 8400 2250
+Wire Wire Line
+	7800 2350 8400 2350
+Wire Wire Line
+	7800 2450 8400 2450
+Wire Wire Line
+	7800 2550 8400 2550
+Wire Bus Line
+	6500 3000 6500 4400
+Wire Wire Line
+	5850 2900 6400 2900
+Wire Wire Line
+	5850 1900 6350 1900
+Wire Wire Line
+	5850 2000 6350 2000
+Wire Wire Line
+	5850 2100 6350 2100
+Wire Wire Line
+	5850 2400 6350 2400
+Wire Wire Line
+	5850 2500 6350 2500
+Wire Wire Line
+	2900 1900 3450 1900
+Wire Wire Line
+	2900 2000 3450 2000
+Wire Wire Line
+	2900 2100 3450 2100
+Wire Wire Line
+	2900 2200 3450 2200
+Wire Wire Line
+	2900 2300 3450 2300
+Wire Wire Line
+	2900 2400 3450 2400
+Wire Wire Line
+	2900 2800 3450 2800
+Wire Wire Line
+	2900 2900 3450 2900
+Wire Wire Line
+	2900 3000 3450 3000
+Wire Wire Line
+	2900 3100 3450 3100
+Wire Wire Line
+	2900 3200 3450 3200
+Wire Wire Line
+	2900 3300 3450 3300
+Wire Wire Line
+	2900 3400 3450 3400
+Wire Wire Line
+	2900 3500 3450 3500
+Wire Wire Line
+	2350 6650 2150 6650
+Connection ~ 2150 6650
+Wire Wire Line
+	9050 3400 9300 3400
+Wire Wire Line
+	9050 3550 9300 3550
+Wire Wire Line
+	9050 3700 9300 3700
+Wire Wire Line
+	9050 3850 9300 3850
+Wire Wire Line
+	9050 4000 9300 4000
+Wire Wire Line
+	9050 4350 9300 4350
+Wire Wire Line
+	9050 4500 9300 4500
+Wire Wire Line
+	9050 4650 9300 4650
+Wire Wire Line
+	9050 4800 9300 4800
+Wire Wire Line
+	9050 4950 9300 4950
+Wire Wire Line
+	9050 4150 9300 4150
+Wire Wire Line
+	2900 4900 2900 5150
+Connection ~ 4300 5750
+Wire Wire Line
+	5050 5750 5050 5550
+Connection ~ 5050 5750
+Wire Wire Line
 	7800 2150 8400 2150
 Wire Wire Line
@@
 Wire Wire Line
 	7800 1150 8400 1150
+Wire Wire Line
+	4700 5050 4700 5150
+Wire Wire Line
+	4700 5150 5050 5150
+Wire Wire Line
+	3050 5750 5450 5750
+$Comp
+L C C5
+U 1 1 5BD344C0
+P 7300 5600
+F 0 "C5" H 7325 5700 50  0000 L CNN
+F 1 "100pF" H 7325 5500 50  0000 L CNN
+F 2 "Capacitors_SMD:C_0603_HandSoldering" H 7338 5450 30  0001 C CNN
+F 3 "" H 7300 5600 60  0000 C CNN
+	1    7300 5600
+	1    0    0    -1
+$EndComp
+$Comp
+L GND #PWR09
+U 1 1 5BD34D49
+P 7100 6000
+F 0 "#PWR09" H 7100 5750 50  0001 C CNN
+F 1 "GND" H 7100 5850 50  0000 C CNN
+F 2 "" H 7100 6000 60  0000 C CNN
+F 3 "" H 7100 6000 60  0000 C CNN
+	1    7100 6000
+	1    0    0    -1
+$EndComp
+Text GLabel 7100 5200 1    60   UnSpc ~ 0
++5V
+Wire Wire Line
+	6900 5450 6900 5350
+Wire Wire Line
+	6900 5350 7300 5350
+Wire Wire Line
+	7300 5350 7300 5450
+Wire Wire Line
+	7100 5200 7100 5350
+Connection ~ 7100 5350
+Wire Wire Line
+	6900 5750 6900 5850
+Wire Wire Line
+	6900 5850 7300 5850
+Wire Wire Line
+	7300 5850 7300 5750
+Wire Wire Line
+	7100 6000 7100 5850
+Connection ~ 7100 5850
+Text Notes 6450 4950 0    118  ~ 24
+IC DECOUPLING
+Text Notes 4900 5000 0    118  ~ 24
+USB POWER
+Wire Wire Line
+	3250 4800 3250 5150
+Connection ~ 3250 5150
 $EndSCHEMATC

Commit message: update
Connections:
- net GND: no longer C3.1, C5.1, P1.2 (P2), P2.1 (VCC), P3.9 (P9), P5.1 (VCC), U1.20 (VDD)
- new net VCC: C3.1, C5.1, P1.2 (P2), P2.1 (VCC), P3.9 (P9), P5.1 (VCC), U1.20 (VDD)

Commit message: another upd
Parts:
- added C6, C7: 10uF, Capacitors_SMD:CP_Elec_4x5.8, symbol CP
- added C8, C9: 100pF, Capacitors_SMD:C_0603_HandSoldering, symbol C
Connections:
- net GND: now also C6.2, C7.2, C8.2, C9.2
- net VCC: now also C6.1, C7.1, C8.1, C9.1
Changed lines of the file:
@@
 Text GLabel 3050 5700 2    60   UnSpc ~ 0
 GND
+$Comp
+L CP C7
+U 1 1 5BDA4749
+P 6550 5600
+F 0 "C7" H 6575 5700 50  0000 L CNN
+F 1 "10uF" H 6575 5500 50  0000 L CNN
+F 2 "Capacitors_SMD:CP_Elec_4x5.8" H 6588 5450 30  0001 C CNN
+F 3 "" H 6550 5600 60  0000 C CNN
+	1    6550 5600
+	1    0    0    -1
+$EndComp
+$Comp
+L CP C6
+U 1 1 5BDA47E5
+P 6200 5600
+F 0 "C6" H 6225 5700 50  0000 L CNN
+F 1 "10uF" H 6225 5500 50  0000 L CNN
+F 2 "Capacitors_SMD:CP_Elec_4x5.8" H 6238 5450 30  0001 C CNN
+F 3 "" H 6200 5600 60  0000 C CNN
+	1    6200 5600
+	1    0    0    -1
+$EndComp
 Wire Wire Line
 	3050 5700 2850 5700
@@
 	7300 5850 7300 5750
 Wire Wire Line
-	6900 5850 7300 5850
+	6200 5850 8050 5850
 Wire Wire Line
 	6900 5750 6900 5850
@@
 	7300 5350 7300 5450
 Wire Wire Line
-	6900 5350 7300 5350
+	6200 5350 8050 5350
 Wire Wire Line
 	6900 5450 6900 5350
@@
 Connection ~ 4300 5800
 Connection ~ 5050 5800
+Wire Wire Line
+	6550 5450 6550 5350
+Connection ~ 6900 5350
+Wire Wire Line
+	6200 5450 6200 5350
+Connection ~ 6550 5350
+Wire Wire Line
+	6550 5750 6550 5850
+Connection ~ 6900 5850
+Wire Wire Line
+	6200 5750 6200 5850
+Connection ~ 6550 5850
+$Comp
+L C C8
+U 1 1 5BDA57EF
+P 7700 5600
+F 0 "C8" H 7725 5700 50  0000 L CNN
+F 1 "100pF" H 7725 5500 50  0000 L CNN
+F 2 "Capacitors_SMD:C_0603_HandSoldering" H 7738 5450 30  0001 C CNN
+F 3 "" H 7700 5600 60  0000 C CNN
+	1    7700 5600
+	1    0    0    -1
+$EndComp
+$Comp
+L C C9
+U 1 1 5BDA5877
+P 8050 5600
+F 0 "C9" H 8075 5700 50  0000 L CNN
+F 1 "100pF" H 8075 5500 50  0000 L CNN
+F 2 "Capacitors_SMD:C_0603_HandSoldering" H 8088 5450 30  0001 C CNN
+F 3 "" H 8050 5600 60  0000 C CNN
+	1    8050 5600
+	1    0    0    -1
+$EndComp
+Wire Wire Line
+	7700 5350 7700 5450
+Connection ~ 7300 5350
+Wire Wire Line
+	8050 5350 8050 5450
+Connection ~ 7700 5350
+Wire Wire Line
+	7700 5850 7700 5750
+Connection ~ 7300 5850
+Wire Wire Line
+	8050 5850 8050 5750
+Connection ~ 7700 5850
 $EndSCHEMATC
