File: AccessB.sch (KiCad schematic (older format))
At the start: 15 parts, among them P1 ICSP, P2 USB_OTG, P3 GPIO, P5 USB_OTG, U1 PIC18(L)F2550-I/SO, Y1 4MHz

Commit message: New update
update
Parts:
- C1, C2, C4, C5, C8, C9: symbol C -> AccessB-rescue:C
- C3, C6, C7: symbol CP -> AccessB-rescue:CP
- P1: symbol CONN_01X05 -> AccessB-rescue:CONN_01X05
- P2, P5: symbol USB_OTG-RESCUE-AccessB -> AccessB-rescue:USB_OTG-RESCUE-AccessB
- P3: symbol CONN_02X15 -> AccessB-rescue:CONN_02X15
- U1: symbol PIC18(L)F2550-I/SO -> AccessB-rescue:PIC18(L)F2550-I_SO
- Y1: symbol Crystal -> AccessB-rescue:Crystal
Changed lines of the file:
@@
-EESchema Schematic File Version 2
-LIBS:AccessB-rescue
-LIBS:switches
-LIBS:power
-LIBS:device
-LIBS:transistors
-LIBS:conn
-LIBS:linear
-LIBS:regul
-LIBS:74xx
-LIBS:cmos4000
-LIBS:adc-dac
-LIBS:memory
-LIBS:xilinx
-LIBS:microcontrollers
-LIBS:dsp
-LIBS:microchip
-LIBS:analog_switches
-LIBS:motorola
-LIBS:texas
-LIBS:intel
-LIBS:audio
-LIBS:interface
-LIBS:digital-audio
-LIBS:philips
-LIBS:display
-LIBS:cypress
-LIBS:siliconi
-LIBS:opto
-LIBS:atmel
-LIBS:contrib
-LIBS:valves
-LIBS:microchip_pic18mcu
-LIBS:brooktre
-LIBS:dc-dc
-LIBS:onsemi
-LIBS:Power_Management
-LIBS:powerint
-LIBS:gennum
-LIBS:Oscillators
-LIBS:Symbols_DCDC-ACDC-Converter_RevC_20Jul2012
-LIBS:Symbols_EN60617_13Mar2013
-LIBS:Symbols_EN60617-10_HF-Radio_DRAFT_12Sep2013
-LIBS:Symbols_ICs-Diskrete_RevD10
-LIBS:Symbols_ICs-Opto_RevB_16Sep2013
-LIBS:Symbols_Microcontroller_Philips-NXP_RevA_06Oct2013
-LIBS:Symbols_Socket-DIN41612_RevA
-LIBS:Symbols_Transformer-Diskrete_RevA
-LIBS:SymbolsSimilarEN60617+oldDIN617-RevE8
-LIBS:74xgxx
-LIBS:ac-dc
-LIBS:actel
-LIBS:Altera
-LIBS:analog_devices
-LIBS:cmos_ieee
-LIBS:diode
-LIBS:elec-unifil
-LIBS:ESD_Protection
-LIBS:ftdi
-LIBS:hc11
-LIBS:ir
-LIBS:Lattice
-LIBS:maxim
-LIBS:microchip_dspic33dsc
-LIBS:microchip_pic10mcu
-LIBS:microchip_pic12mcu
-LIBS:microchip_pic16mcu
-LIBS:microchip_pic32mcu
-LIBS:motor_drivers
-LIBS:msp430
-LIBS:nordicsemi
-LIBS:nxp_armmcu
-LIBS:pspice
-LIBS:references
-LIBS:relays
-LIBS:rfcom
-LIBS:sensors
-LIBS:silabs
-LIBS:stm8
-LIBS:stm32
-LIBS:supertex
-LIBS:transf
-LIBS:ttl_ieee
-LIBS:video
-LIBS:Xicor
-LIBS:Zilog
-LIBS:Microchip MCP1306
+EESchema Schematic File Version 4
 LIBS:AccessB-cache
-EELAYER 25 0
+EELAYER 26 0
 EELAYER END
 $Descr A4 11693 8268
@@
 $EndDescr
 $Comp
-L USB_OTG-RESCUE-AccessB P2
+L AccessB-rescue:USB_OTG-RESCUE-AccessB P2
 U 1 1 562726A7
 P 4200 5350
@@
 $EndComp
 $Comp
-L C C1
+L AccessB-rescue:C C1
 U 1 1 5629BFE7
 P 1650 3400
@@
 $EndComp
 $Comp
-L C C2
+L AccessB-rescue:C C2
 U 1 1 5629C07C
 P 2250 3400
@@
 $EndComp
 $Comp
-L C C4
+L AccessB-rescue:C C4
 U 1 1 5629C0B9
 P 6800 3050
@@
 $EndComp
 $Comp
-L CP C3
+L AccessB-rescue:CP C3
 U 1 1 5629C0F8
 P 6900 5600
@@
 $EndComp
 $Comp
-L CONN_01X05 P1
+L AccessB-rescue:CONN_01X05 P1
 U 1 1 5629C382
 P 2000 5400
@@
 $EndComp
 $Comp
-L PIC18(L)F2550-I/SO U1
+L AccessB-rescue:PIC18(L)F2550-I_SO U1
 U 1 1 562721CB
 P 4650 2700
@@
 $EndSheet
 $Comp
-L GND #PWR01
+L power:GND #PWR01
 U 1 1 5632DC45
 P 2850 5800
@@
 $EndComp
 $Comp
-L Crystal Y1
+L AccessB-rescue:Crystal Y1
 U 1 1 5632E118
 P 1950 2900
@@
 $EndComp
 $Comp
-L GND #PWR02
+L power:GND #PWR02
 U 1 1 56330810
 P 1950 3900
@@
 $EndComp
 $Comp
-L PWR_FLAG #FLG03
+L power:PWR_FLAG #FLG03
 U 1 1 56332B13
 P 2850 5600
@@
 $EndComp
 $Comp
-L GND #PWR04
+L power:GND #PWR04
 U 1 1 56332E46
 P 4600 4000
@@
 GND
 $Comp
-L GND #PWR05
+L power:GND #PWR05
 U 1 1 56367ADB
 P 3750 5850
@@
 GPIO0/RE3
 $Comp
-L GND #PWR06
+L power:GND #PWR06
 U 1 1 5636AE18
 P 6800 3400
@@
 GND
 $Comp
-L CONN_02X15 P3
+L AccessB-rescue:CONN_02X15 P3
 U 1 1 56376D9B
 P 8650 1850
@@
 GND
 $Comp
-L USB_OTG-RESCUE-AccessB P5
+L AccessB-rescue:USB_OTG-RESCUE-AccessB P5
 U 1 1 592BE443
 P 5350 5350
@@
 NoConn ~ 5050 5250
 $Comp
-L VCC #PWR07
+L power:VCC #PWR07
 U 1 1 592D4E49
 P 2900 4900
@@
 	7700 2050 7800 2150
 $Comp
-L C C5
+L AccessB-rescue:C C5
 U 1 1 5BD344C0
 P 7300 5600
@@
 $EndComp
 $Comp
-L GND #PWR08
+L power:GND #PWR08
 U 1 1 5BD34D49
 P 7100 6000
@@
 USB POWER
 $Comp
-L PWR_FLAG #FLG09
+L power:PWR_FLAG #FLG09
 U 1 1 5BD3BDCF
 P 3250 4900
@@
 GND
 $Comp
-L CP C7
+L AccessB-rescue:CP C7
 U 1 1 5BDA4749
 P 6550 5600
@@
 $EndComp
 $Comp
-L CP C6
+L AccessB-rescue:CP C6
 U 1 1 5BDA47E5
 P 6200 5600
@@
 	7300 5850 7300 5750
 Wire Wire Line
-	6200 5850 8050 5850
+	6200 5850 6550 5850
 Wire Wire Line
 	6900 5750 6900 5850
@@
 	7300 5350 7300 5450
 Wire Wire Line
-	6200 5350 8050 5350
+	6200 5350 6550 5350
 Wire Wire Line
 	6900 5450 6900 5350
@@
 	7700 4400 2800 4400
 Wire Bus Line
-	2800 4400 2800 2900
-Wire Bus Line
-	6450 1000 6450 2400
-Wire Bus Line
-	7700 1000 7700 4400
-Wire Bus Line
 	2800 1000 9800 1000
-Wire Bus Line
-	2800 1000 2800 2300
 Wire Wire Line
 	6800 3200 6800 3400
@@
 	3450 2500 1650 2500
 Wire Wire Line
-	3750 5550 3750 5850
+	3750 5550 3750 5800
 Wire Wire Line
 	3900 5550 3750 5550
 Wire Wire Line
-	2900 5150 3900 5150
+	2900 5150 3050 5150
 Wire Wire Line
 	4650 1600 4650 1400
 Wire Wire Line
-	2850 5600 2850 5800
+	2850 5600 2850 5700
 Connection ~ 4600 4000
 Wire Wire Line
 	4650 4000 4650 3800
 Wire Wire Line
-	4550 4000 4650 4000
+	4550 4000 4600 4000
 Wire Wire Line
 	4550 3800 4550 4000
@@
 	2250 3750 2250 3550
 Wire Wire Line
-	1650 3750 2250 3750
+	1650 3750 1950 3750
 Wire Wire Line
 	1650 3550 1650 3750
@@
 	2250 2900 2100 2900
 Wire Wire Line
-	2250 2600 2250 3250
+	2250 2600 2250 2900
 Wire Wire Line
 	1650 2900 1800 2900
 Wire Wire Line
-	1650 2500 1650 3250
+	1650 2500 1650 2900
 Wire Wire Line
 	3050 5000 3050 5150
@@
 	5450 5750 5450 5800
 Wire Wire Line
-	5450 5800 3750 5800
+	5450 5800 5050 5800
 Connection ~ 3750 5800
 Wire Wire Line
@@
 Connection ~ 6550 5850
 $Comp
-L C C8
+L AccessB-rescue:C C8
 U 1 1 5BDA57EF
 P 7700 5600
@@
 $EndComp
 $Comp
-L C C9
+L AccessB-rescue:C C9
 U 1 1 5BDA5877
 P 8050 5600
@@
 	8050 5850 8050 5750
 Connection ~ 7700 5850
+Wire Wire Line
+	2850 5700 2850 5800
+Wire Wire Line
+	7100 5850 7300 5850
+Wire Wire Line
+	7100 5350 7300 5350
+Wire Wire Line
+	2250 2900 2250 3250
+Wire Wire Line
+	1650 2900 1650 3250
+Wire Wire Line
+	4600 4000 4650 4000
+Wire Wire Line
+	1950 3750 2250 3750
+Wire Wire Line
+	3050 5150 3250 5150
+Wire Wire Line
+	3250 5150 3900 5150
+Wire Wire Line
+	3750 5800 3750 5850
+Wire Wire Line
+	4300 5800 3750 5800
+Wire Wire Line
+	5050 5800 4300 5800
+Wire Wire Line
+	6900 5350 7100 5350
+Wire Wire Line
+	6550 5350 6900 5350
+Wire Wire Line
+	6900 5850 7100 5850
+Wire Wire Line
+	6550 5850 6900 5850
+Wire Wire Line
+	7300 5350 7700 5350
+Wire Wire Line
+	7700 5350 8050 5350
+Wire Wire Line
+	7300 5850 7700 5850
+Wire Wire Line
+	7700 5850 8050 5850
+Wire Bus Line
+	6450 1000 6450 2400
+Wire Bus Line
+	2800 1000 2800 2300
+Wire Bus Line
+	2800 2900 2800 4400
+Wire Bus Line
+	7700 1000 7700 4400
 $EndSCHEMATC

Commit message: Update
Some reworking....
Connections:
- net GPIO11/RA5_VLS: now also P3.4 (P4); no longer P3.10 (P10)
- net GPIO12/RB0_VLS: now also P3.6 (P6); no longer P3.8 (P8)
- net GPIO13/RB1_VLS: now also P3.2 (P2); no longer P3.6 (P6)
- net GPIO4/RC6_VLS: now also P3.10 (P10); no longer P3.4 (P4)
- net GPIO5/RC7_VLS: now also P3.8 (P8); no longer P3.2 (P2)
Changed lines of the file:
@@
 Text Label 8400 2550 2    60   ~ 0
 GPIO19/RB7
+Text Label 8900 1550 0    60   ~ 0
+GPIO4/RC6_VLS
+Text Label 8900 1450 0    60   ~ 0
+GPIO5/RC7_VLS
 Text Label 8900 1250 0    60   ~ 0
-GPIO4/RC6_VLS
+GPIO11/RA5_VLS
+Text Label 8900 1350 0    60   ~ 0
+GPIO12/RB0_VLS
 Text Label 8900 1150 0    60   ~ 0
-GPIO5/RC7_VLS
-Text Label 8900 1550 0    60   ~ 0
-GPIO11/RA5_VLS
-Text Label 8900 1450 0    60   ~ 0
-GPIO12/RB0_VLS
-Text Label 8900 1350 0    60   ~ 0
 GPIO13/RB1_VLS
 Text Label 8400 1550 2    60   ~ 0

Commit message: sdf
df
Connections:
- net D+/RC5 renamed D+
- net D-/RC4 renamed D-
Changed lines of the file:
@@
 NoConn ~ 3900 5450
 Text Label 3900 5250 2    60   ~ 0
-D-/RC4
+D-
 Text Label 3900 5350 2    60   ~ 0
-D+/RC5
+D+
 Text Label 1800 5600 2    60   ~ 0
 GPIO18/RB6
@@
 Text Label 5850 2100 0    60   ~ 0
 GPIO3/RC2
-Text Label 5850 2200 0    60   ~ 0
-D-/RC4
 Text Label 5850 2300 0    60   ~ 0
-D+/RC5
+D+
 Text Label 5850 2400 0    60   ~ 0
 GPIO4/RC6
@@
 	7700 5850 8050 5850
 Wire Bus Line
+	7700 1000 7700 4400
+Wire Bus Line
+	2800 2900 2800 4400
+Wire Bus Line
+	2800 1000 2800 2300
+Wire Bus Line
 	6450 1000 6450 2400
-Wire Bus Line
-	2800 1000 2800 2300
-Wire Bus Line
-	2800 2900 2800 4400
-Wire Bus Line
-	7700 1000 7700 4400
+Text Label 5850 2200 0    60   ~ 0
+D-
 $EndSCHEMATC
